File: lab4/exercise1/exercise1.kicad_sch (KiCad schematic)
At the start: 6 parts, among them SW1 SW_SPDT

Commit message: update
Other:
- title: (none) -> Exercise 1
Changed lines of the file:
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@@
 (kicad_sch (version 20211123) (generator eeschema)
   (paper "A4")
+  (title_block
+    (title "Exercise 1")
+    (date "2023-01-27")
+  )
   (junction (at 102.87 87.63) (diameter 0) (color 0 0 0 0)
   )
@@
   (symbol (lib_id "Switch:SW_SPDT") (at 92.71 67.31 0) (unit 1)
     (in_bom yes) (on_board yes) (fields_autoplaced)
-    (property "Reference" "SW1" (id 0) (at 92.71 59.69 0))
-    (property "Value" "SW_SPDT" (id 1) (at 92.71 62.23 0))
+    (property "Reference" "SW1" (id 0) (at 92.71 62.23 0))
+    (property "Value" "SW_SPDT" (id 1) (at 92.71 62.23 0)
+      (effects (font (size 1.27 1.27)) hide)
+    )
     (property "Footprint" "" (id 2) (at 92.71 67.31 0)
       (effects (font (size 1.27 1.27)) hide)
