File: lab4/exercise2/exercise2.kicad_sch (KiCad schematic)
At the start: 10 parts, among them J1 9V, U1 NE555D

Commit message: update
Other:
- title: (none) -> Exercise 2
Changed lines of the file:
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@@
 (kicad_sch (version 20211123) (generator eeschema)
   (paper "A4")
+  (title_block
+    (title "Exercise 2")
+    (date "2023-01-27")
+  )
   (junction (at 172.72 92.71) (diameter 0) (color 0 0 0 0)
   )
